Commit message: update my_robot.xacro

File: project_2/catkin_ws/src/my_robot/urdf/my_robot.xacro (robot description, xacro)
@@ -30,16 +30,4 @@
       </geometry>
     </visual>
-    <collision name='back_caster_collision'>
-      <origin xyz="-0.15 0 -0.05" rpy=" 0 0 0"/>
-      <geometry>
-        <sphere radius="0.0499"/>
-      </geometry>
-    </collision>
-    <visual name='back_caster_visual'>
-      <origin xyz="-0.15 0 -0.05" rpy=" 0 0 0"/>
-      <geometry>
-        <sphere radius="0.05"/>
-      </geometry>
-    </visual>
     <collision name='front_caster_collision'>
       <origin xyz="0.15 0 -0.05" rpy=" 0 0 0"/>
@@ -55,3 +43,27 @@
     </visual>
   </link>
+  <link name='left_wheel'>
+    <pose>0 -0.15 0 0 0 0</pose>
+    <inertial>
+      <mass value="5.0"/>
+      <origin xyz="0.0 0 0" rpy=" 0 0 0"/>
+      <inertia
+          ixx="0.1" ixy="0" ixz="0"
+          iyy="0.1" iyz="0"
+          izz="0.1"
+      />
+    </inertial>
+    <collision name='left_wheel_collision'>
+      <origin xyz="0 0 0" rpy=" 0 1.5707 1.5707"/>
+      <geometry>
+        <cylinder radius=".1" length="0.05"/>
+      </geometry>
+    </collision>
+    <visual name='left_wheel_visual'>
+      <origin xyz="0 0 0" rpy=" 0 1.5707 1.5707"/>
+      <geometry>
+        <cylinder radius=".1" length="0.05"/>
+      </geometry>
+    </visual>
+  </link>
 </robot>

Commit message: update left_wheel

File: project_2/catkin_ws/src/my_robot/urdf/my_robot.xacro (robot description, xacro)
@@ -47,10 +47,9 @@
     <inertial>
       <mass value="5.0"/>
-      <origin xyz="0.0 0 0" rpy=" 0 0 0"/>
+      <origin xyz="0.0 0 0" rpy=" 0 1.5707 1.5707"/>
       <inertia
           ixx="0.1" ixy="0" ixz="0"
           iyy="0.1" iyz="0"
-          izz="0.1"
-      />
+          izz="0.1"/>
     </inertial>
     <collision name='left_wheel_collision'>

Commit message: update .xacro

File: project_2/catkin_ws/src/my_robot/urdf/my_robot.xacro (robot description, xacro)
@@ -44,4 +44,27 @@
   </link>
   <link name='left_wheel'>
+    <pose>0 0.15 0 0 0 0</pose>
+    <inertial>
+      <mass value="5.0"/>
+      <origin xyz="0.0 0 0" rpy=" 0 1.5707 1.5707"/>
+      <inertia
+          ixx="0.1" ixy="0" ixz="0"
+          iyy="0.1" iyz="0"
+          izz="0.1"/>
+    </inertial>
+    <collision name='left_wheel_collision'>
+      <origin xyz="0 0 0" rpy=" 0 1.5707 1.5707"/>
+      <geometry>
+        <cylinder radius=".1" length="0.05"/>
+      </geometry>
+    </collision>
+    <visual name='left_wheel_visual'>
+      <origin xyz="0 0 0" rpy=" 0 1.5707 1.5707"/>
+      <geometry>
+        <cylinder radius=".1" length="0.05"/>
+      </geometry>
+    </visual>
+  </link>
+  <link name='right_wheel'>
     <pose>0 -0.15 0 0 0 0</pose>
     <inertial>
@@ -66,3 +89,19 @@
     </visual>
   </link>
+  <joint type="continuous" name="left_wheel_hinge">
+    <origin xyz="0 0.15 0" rpy="0 0 0"/>
+    <child link="left_wheel"/>
+    <parent link="chassis"/>
+    <axis xyz="0 1 0" rpy="0 0 0"/>
+    <limit effort="10000" velocity="1000"/>
+    <dynamics damping="1.0" friction="1.0"/>
+  </joint>
+  <joint type="continuous" name="right_wheel_hinge">
+    <origin xyz="0 -0.15 0" rpy="0 0 0"/>
+    <child link="right_wheel"/>
+    <parent link="chassis"/>
+    <axis xyz="0 1 0" rpy="0 0 0"/>
+    <limit effort="10000" velocity="1000"/>
+    <dynamics damping="1.0" friction="1.0"/>
+  </joint>
 </robot>

Commit message: camera added to .xacro

File: project_2/catkin_ws/src/my_robot/urdf/my_robot.xacro (robot description, xacro)
@@ -105,3 +105,32 @@
     <dynamics damping="1.0" friction="1.0"/>
   </joint>
+  <link name='camera'>
+    <pose>0 -0.15 0 0 0 0</pose>
+    <inertial>
+      <mass value=".1"/>
+      <origin xyz="0.2 0 0" rpy=" 0 0 0"/>
+      <inertia
+          ixx="1e-6" ixy="0" ixz="0"
+          iyy="1e-6" iyz="0"
+          izz="1e-6"/>
+    </inertial>
+    <collision name='camera_collision'>
+      <origin xyz="0.2 0 0" rpy=" 0 0 0"/>
+      <geometry>
+        <box size=".05 .05 .05"/>
+      </geometry>
+    </collision>
+    <visual name='camera_visual'>
+      <origin xyz="0.2 0 0" rpy=" 0 0 0"/>
+      <geometry>
+        <box size=".05 .05 .05"/>
+      </geometry>
+    </visual>
+  </link>
+  <joint type="fixed" name="camera_joint">
+    <origin xyz=".2 0 0" rpy="0 0 0"/>
+    <child link="camera"/>
+    <parent link="chassis"/>
+    <axis xyz="0 1 0" rpy="0 0 0"/>
+  </joint>
 </robot>

Commit message: update .xacro for camera

File: project_2/catkin_ws/src/my_robot/urdf/my_robot.xacro (robot description, xacro)
@@ -89,4 +89,27 @@
     </visual>
   </link>
+  <link name='camera'>
+    <pose> 0.2 0 0 0 0 0</pose>
+    <inertial>
+      <mass value=".1"/>
+      <origin xyz="0 0 0" rpy=" 0 0 0"/>
+      <inertia
+          ixx="1e-6" ixy="0" ixz="0"
+          iyy="1e-6" iyz="0"
+          izz="1e-6"/>
+    </inertial>
+    <collision name='camera_collision'>
+      <origin xyz="0 0 0" rpy=" 0 0 0"/>
+      <geometry>
+        <box size=".05 .05 .05"/>
+      </geometry>
+    </collision>
+    <visual name='camera_visual'>
+      <origin xyz="0 0 0" rpy=" 0 0 0"/>
+      <geometry>
+        <box size=".05 .05 .05"/>
+      </geometry>
+    </visual>
+  </link>
   <joint type="continuous" name="left_wheel_hinge">
     <origin xyz="0 0.15 0" rpy="0 0 0"/>
@@ -105,32 +128,9 @@
     <dynamics damping="1.0" friction="1.0"/>
   </joint>
-  <link name='camera'>
-    <pose>0 -0.15 0 0 0 0</pose>
-    <inertial>
-      <mass value=".1"/>
-      <origin xyz="0.2 0 0" rpy=" 0 0 0"/>
-      <inertia
-          ixx="1e-6" ixy="0" ixz="0"
-          iyy="1e-6" iyz="0"
-          izz="1e-6"/>
-    </inertial>
-    <collision name='camera_collision'>
-      <origin xyz="0.2 0 0" rpy=" 0 0 0"/>
-      <geometry>
-        <box size=".05 .05 .05"/>
-      </geometry>
-    </collision>
-    <visual name='camera_visual'>
-      <origin xyz="0.2 0 0" rpy=" 0 0 0"/>
-      <geometry>
-        <box size=".05 .05 .05"/>
-      </geometry>
-    </visual>
-  </link>
   <joint type="fixed" name="camera_joint">
-    <origin xyz=".2 0 0" rpy="0 0 0"/>
+    <origin xyz="0.2 0 0" rpy="0 0 0"/>
     <child link="camera"/>
     <parent link="chassis"/>
-    <axis xyz="0 1 0" rpy="0 0 0"/>
+    <axis xyz="1 1 1" rpy="0 0 0"/>
   </joint>
 </robot>

Commit message: update .xacro and .gitignore

File: project_2/catkin_ws/src/my_robot/urdf/my_robot.xacro (robot description, xacro)
@@ -112,4 +112,27 @@
     </visual>
   </link>
+  <link name='hokuyo'>
+    <pose>0.15 0 .1 0 0 0</pose>
+    <inertial>
+      <mass value="1e-5"/>
+      <origin xyz="0 0 0" rpy=" 0 0 0"/>
+      <inertia
+          ixx="1e-6" ixy="0" ixz="0"
+          iyy="1e-6" iyz="0"
+          izz="1e-6"/>
+    </inertial>
+    <collision name='hokuyo_collision'>
+      <origin xyz="0 0 0" rpy=" 0 0 0"/>
+      <geometry>
+        <box size=".1 .1 .1"/>
+      </geometry>
+    </collision>
+    <visual name='hokuyo_visual'>
+      <origin xyz="0 0 0" rpy=" 0 0 0"/>
+      <geometry>
+        <filename="package://my_robot/meshes/hokuyo.dae"/>
+      </geometry>
+    </visual>
+  </link>
   <joint type="continuous" name="left_wheel_hinge">
     <origin xyz="0 0.15 0" rpy="0 0 0"/>
@@ -134,3 +157,9 @@
     <axis xyz="1 1 1" rpy="0 0 0"/>
   </joint>
+  <joint type="fixed" name="hokuyo_joint">
+    <origin xyz="0.15 0 .1" rpy="0 0 0"/>
+    <child link="hokuyo"/>
+    <parent link="chassis"/>
+    <axis xyz="1 1 1" rpy="0 0 0"/>
+  </joint>
 </robot>

Commit message: update .xacro file

File: project_2/catkin_ws/src/my_robot/urdf/my_robot.xacro (robot description, xacro)
@@ -111,4 +111,7 @@
       </geometry>
     </visual>
+    <gazebo reference="left_wheel">
+        <material>Gazebo/Red</material>
+    </gazebo>
   </link>
   <link name='hokuyo'>

Commit message: update .xacro

File: project_2/catkin_ws/src/my_robot/urdf/my_robot.xacro (robot description, xacro)
@@ -76,5 +76,5 @@
           izz="0.1"/>
     </inertial>
-    <collision name='left_wheel_collision'>
+    <collision name='right_wheel_collision'>
       <origin xyz="0 0 0" rpy=" 0 1.5707 1.5707"/>
       <geometry>
@@ -82,5 +82,5 @@
       </geometry>
     </collision>
-    <visual name='left_wheel_visual'>
+    <visual name='right_wheel_visual'>
       <origin xyz="0 0 0" rpy=" 0 1.5707 1.5707"/>
       <geometry>
@@ -111,10 +111,7 @@
       </geometry>
     </visual>
-    <gazebo reference="left_wheel">
-        <material>Gazebo/Red</material>
-    </gazebo>
   </link>
   <link name='hokuyo'>
-    <pose>0.15 0 .1 0 0 0</pose>
+    <pose>0 0 0 0 0 0</pose>
     <inertial>
       <mass value="1e-5"/>
@@ -134,8 +131,14 @@
       <origin xyz="0 0 0" rpy=" 0 0 0"/>
       <geometry>
-        <filename="package://my_robot/meshes/hokuyo.dae"/>
+        <mesh filename="package://my_robot/meshes/hokuyo.dae"/>
       </geometry>
     </visual>
-  </link>
+</link>
+<joint type="fixed" name="hokuyo_joint">
+  <origin xyz="0.15 0 .1" rpy="0 0 0"/>
+  <child link="hokuyo"/>
+  <parent link="chassis"/>
+  <axis xyz="1 1 1" rpy="0 0 0"/>
+</joint>
   <joint type="continuous" name="left_wheel_hinge">
     <origin xyz="0 0.15 0" rpy="0 0 0"/>
@@ -160,9 +163,15 @@
     <axis xyz="1 1 1" rpy="0 0 0"/>
   </joint>
-  <joint type="fixed" name="hokuyo_joint">
-    <origin xyz="0.15 0 .1" rpy="0 0 0"/>
-    <child link="hokuyo"/>
-    <parent link="chassis"/>
-    <axis xyz="1 1 1" rpy="0 0 0"/>
-  </joint>
+  <gazebo reference="camera">
+      <material>Gazebo/Red</material>
+  </gazebo>
+  <gazebo reference="left_wheel">
+      <material>Gazebo/Yellow</material>
+  </gazebo>
+  <gazebo reference="right_wheel">
+      <material>Gazebo/Yellow</material>
+  </gazebo>
+  <gazebo reference="chassis">
+      <material>Gazebo/Green</material>
+  </gazebo>
 </robot>

Commit message: update urdf and launch files

File: project_2/catkin_ws/src/my_robot/urdf/my_robot.xacro (robot description, xacro)
@@ -1,4 +1,5 @@
 <?xml version='1.0'?>
 <robot name="my_robot" xmlns:xacro="http://www.ros.org/wiki/xacro">
+  <xacro:include filename="$(find my_robot)/urdf/my_robot.gazebo" />
   <link name="robot_footprint"></link>
   <joint name="robot_footprint_joint" type="fixed">
@@ -76,5 +77,5 @@
           izz="0.1"/>
     </inertial>
-    <collision name='right_wheel_collision'>
+    <collision name='left_wheel_collision'>
       <origin xyz="0 0 0" rpy=" 0 1.5707 1.5707"/>
       <geometry>
@@ -82,5 +83,5 @@
       </geometry>
     </collision>
-    <visual name='right_wheel_visual'>
+    <visual name='left_wheel_visual'>
       <origin xyz="0 0 0" rpy=" 0 1.5707 1.5707"/>
       <geometry>
@@ -111,7 +112,10 @@
       </geometry>
     </visual>
+    <gazebo reference="left_wheel">
+        <material>Gazebo/Red</material>
+    </gazebo>
   </link>
   <link name='hokuyo'>
-    <pose>0 0 0 0 0 0</pose>
+    <pose>0.15 0 .1 0 0 0</pose>
     <inertial>
       <mass value="1e-5"/>
@@ -131,14 +135,8 @@
       <origin xyz="0 0 0" rpy=" 0 0 0"/>
       <geometry>
-        <mesh filename="package://my_robot/meshes/hokuyo.dae"/>
+        <filename="package://my_robot/meshes/hokuyo.dae"/>
       </geometry>
     </visual>
-</link>
-<joint type="fixed" name="hokuyo_joint">
-  <origin xyz="0.15 0 .1" rpy="0 0 0"/>
-  <child link="hokuyo"/>
-  <parent link="chassis"/>
-  <axis xyz="1 1 1" rpy="0 0 0"/>
-</joint>
+  </link>
   <joint type="continuous" name="left_wheel_hinge">
     <origin xyz="0 0.15 0" rpy="0 0 0"/>
@@ -163,15 +161,9 @@
     <axis xyz="1 1 1" rpy="0 0 0"/>
   </joint>
-  <gazebo reference="camera">
-      <material>Gazebo/Red</material>
-  </gazebo>
-  <gazebo reference="left_wheel">
-      <material>Gazebo/Yellow</material>
-  </gazebo>
-  <gazebo reference="right_wheel">
-      <material>Gazebo/Yellow</material>
-  </gazebo>
-  <gazebo reference="chassis">
-      <material>Gazebo/Green</material>
-  </gazebo>
+  <joint type="fixed" name="hokuyo_joint">
+    <origin xyz="0.15 0 .1" rpy="0 0 0"/>
+    <child link="hokuyo"/>
+    <parent link="chassis"/>
+    <axis xyz="1 1 1" rpy="0 0 0"/>
+  </joint>
 </robot>

Commit message: update .xacro

File: project_2/catkin_ws/src/my_robot/urdf/my_robot.xacro (robot description, xacro)
@@ -43,4 +43,16 @@
       </geometry>
     </visual>
+    <collision name='back_caster_collision'>
+      <origin xyz="-0.15 0 -0.05" rpy=" 0 0 0"/>
+      <geometry>
+        <sphere radius="0.0499"/>
+      </geometry>
+    </collision>
+    <visual name='back_caster_visual'>
+      <origin xyz="-0.15 0 -0.05" rpy=" 0 0 0"/>
+      <geometry>
+        <sphere radius="0.05"/>
+      </geometry>
+    </visual>
   </link>
   <link name='left_wheel'>
@@ -77,5 +89,5 @@
           izz="0.1"/>
     </inertial>
-    <collision name='left_wheel_collision'>
+    <collision name='right_wheel_collision'>
       <origin xyz="0 0 0" rpy=" 0 1.5707 1.5707"/>
       <geometry>
@@ -83,5 +95,5 @@
       </geometry>
     </collision>
-    <visual name='left_wheel_visual'>
+    <visual name='right_wheel_visual'>
       <origin xyz="0 0 0" rpy=" 0 1.5707 1.5707"/>
       <geometry>
@@ -112,7 +124,4 @@
       </geometry>
     </visual>
-    <gazebo reference="left_wheel">
-        <material>Gazebo/Red</material>
-    </gazebo>
   </link>
   <link name='hokuyo'>
@@ -135,5 +144,5 @@
       <origin xyz="0 0 0" rpy=" 0 0 0"/>
       <geometry>
-        <filename="package://my_robot/meshes/hokuyo.dae"/>
+        <mesh filename="package://my_robot/meshes/hokuyo.dae"/>
       </geometry>
     </visual>
@@ -167,3 +176,15 @@
     <axis xyz="1 1 1" rpy="0 0 0"/>
   </joint>
+  <gazebo reference="left_wheel">
+      <material>Gazebo/Yellow</material>
+  </gazebo>
+  <gazebo reference="right_wheel">
+      <material>Gazebo/Yellow</material>
+  </gazebo>
+  <gazebo reference="chassis">
+      <material>Gazebo/Green</material>
+  </gazebo>
+    <gazebo reference="camera">
+        <material>Gazebo/Red</material>
+    </gazebo>
 </robot>
