Commit message: update project 2

File: project_2/catkin_ws/src/my_robot/urdf/my_robot.xacro (robot description, xacro)
@@ -11,5 +11,5 @@
     <pose>0 0 0.1 0 0 0</pose>
     <inertial>
-      <mass value="15.0"/>
+      <mass value="5.0"/>
       <origin xyz="0.0 0 0" rpy=" 0 0 0"/>
       <inertia
@@ -22,5 +22,5 @@
       <origin xyz="0 0 0" rpy=" 0 0 0"/>
       <geometry>
-        <box size=".4 .2 .1"/>
+        <box size=".25 .4 .1"/>
       </geometry>
     </collision>
@@ -28,5 +28,17 @@
       <origin xyz="0 0 0" rpy=" 0 0 0"/>
       <geometry>
-        <box size=".4 .2 .1"/>
+        <box size=".25 .4 .1"/>
+      </geometry>
+    </visual>
+    <collision name='back_caster_collision'>
+      <origin xyz="-0.15 0 -0.05" rpy=" 0 0 0"/>
+      <geometry>
+        <sphere radius="0.03"/>
+      </geometry>
+    </collision>
+    <visual name='back_caster_visual'>
+      <origin xyz="-0.15 0 -0.05" rpy=" 0 0 0"/>
+      <geometry>
+        <sphere radius="0.03"/>
       </geometry>
     </visual>
@@ -34,5 +46,5 @@
       <origin xyz="0.15 0 -0.05" rpy=" 0 0 0"/>
       <geometry>
-        <sphere radius="0.0499"/>
+        <sphere radius="0.03"/>
       </geometry>
     </collision>
@@ -40,24 +52,12 @@
       <origin xyz="0.15 0 -0.05" rpy=" 0 0 0"/>
       <geometry>
-        <sphere radius="0.05"/>
-      </geometry>
-    </visual>
-    <collision name='back_caster_collision'>
-      <origin xyz="-0.15 0 -0.05" rpy=" 0 0 0"/>
-      <geometry>
-        <sphere radius="0.0499"/>
-      </geometry>
-    </collision>
-    <visual name='back_caster_visual'>
-      <origin xyz="-0.15 0 -0.05" rpy=" 0 0 0"/>
-      <geometry>
-        <sphere radius="0.05"/>
+        <sphere radius="0.03"/>
       </geometry>
     </visual>
   </link>
-  <link name='left_wheel'>
-    <pose>0 0.15 0 0 0 0</pose>
+ <link name='left_wheel'>
+    <pose>0 0 0 0 0 0</pose>
     <inertial>
-      <mass value="5.0"/>
+      <mass value="3.0"/>
       <origin xyz="0.0 0 0" rpy=" 0 1.5707 1.5707"/>
       <inertia
@@ -69,5 +69,5 @@
       <origin xyz="0 0 0" rpy=" 0 1.5707 1.5707"/>
       <geometry>
-        <cylinder radius=".1" length="0.05"/>
+        <cylinder radius=".08" length="0.025"/>
       </geometry>
     </collision>
@@ -75,116 +75,116 @@
       <origin xyz="0 0 0" rpy=" 0 1.5707 1.5707"/>
       <geometry>
-        <cylinder radius=".1" length="0.05"/>
+        <cylinder radius=".08" length="0.025"/>
       </geometry>
     </visual>
-  </link>
-  <link name='right_wheel'>
-    <pose>0 -0.15 0 0 0 0</pose>
-    <inertial>
-      <mass value="5.0"/>
-      <origin xyz="0.0 0 0" rpy=" 0 1.5707 1.5707"/>
-      <inertia
-          ixx="0.1" ixy="0" ixz="0"
-          iyy="0.1" iyz="0"
-          izz="0.1"/>
-    </inertial>
-    <collision name='right_wheel_collision'>
-      <origin xyz="0 0 0" rpy=" 0 1.5707 1.5707"/>
-      <geometry>
-        <cylinder radius=".1" length="0.05"/>
-      </geometry>
-    </collision>
-    <visual name='right_wheel_visual'>
-      <origin xyz="0 0 0" rpy=" 0 1.5707 1.5707"/>
-      <geometry>
-        <cylinder radius=".1" length="0.05"/>
-      </geometry>
-    </visual>
-  </link>
-  <link name='camera'>
-    <pose> 0.2 0 0 0 0 0</pose>
-    <inertial>
-      <mass value=".1"/>
-      <origin xyz="0 0 0" rpy=" 0 0 0"/>
-      <inertia
-          ixx="1e-6" ixy="0" ixz="0"
-          iyy="1e-6" iyz="0"
-          izz="1e-6"/>
-    </inertial>
-    <collision name='camera_collision'>
-      <origin xyz="0 0 0" rpy=" 0 0 0"/>
-      <geometry>
-        <box size=".05 .05 .05"/>
-      </geometry>
-    </collision>
-    <visual name='camera_visual'>
-      <origin xyz="0 0 0" rpy=" 0 0 0"/>
-      <geometry>
-        <box size=".05 .05 .05"/>
-      </geometry>
-    </visual>
-  </link>
-  <link name='hokuyo'>
-    <pose>0.15 0 .1 0 0 0</pose>
-    <inertial>
-      <mass value="1e-5"/>
-      <origin xyz="0 0 0" rpy=" 0 0 0"/>
-      <inertia
-          ixx="1e-6" ixy="0" ixz="0"
-          iyy="1e-6" iyz="0"
-          izz="1e-6"/>
-    </inertial>
-    <collision name='hokuyo_collision'>
-      <origin xyz="0 0 0" rpy=" 0 0 0"/>
-      <geometry>
-        <box size=".1 .1 .1"/>
-      </geometry>
-    </collision>
-    <visual name='hokuyo_visual'>
-      <origin xyz="0 0 0" rpy=" 0 0 0"/>
-      <geometry>
-        <mesh filename="package://my_robot/meshes/hokuyo.dae"/>
-      </geometry>
-    </visual>
-  </link>
-  <joint type="continuous" name="left_wheel_hinge">
-    <origin xyz="0 0.15 0" rpy="0 0 0"/>
-    <child link="left_wheel"/>
-    <parent link="chassis"/>
-    <axis xyz="0 1 0" rpy="0 0 0"/>
-    <limit effort="10000" velocity="1000"/>
-    <dynamics damping="1.0" friction="1.0"/>
-  </joint>
-  <joint type="continuous" name="right_wheel_hinge">
-    <origin xyz="0 -0.15 0" rpy="0 0 0"/>
-    <child link="right_wheel"/>
-    <parent link="chassis"/>
-    <axis xyz="0 1 0" rpy="0 0 0"/>
-    <limit effort="10000" velocity="1000"/>
-    <dynamics damping="1.0" friction="1.0"/>
-  </joint>
-  <joint type="fixed" name="camera_joint">
-    <origin xyz="0.2 0 0" rpy="0 0 0"/>
-    <child link="camera"/>
-    <parent link="chassis"/>
-    <axis xyz="1 1 1" rpy="0 0 0"/>
-  </joint>
-  <joint type="fixed" name="hokuyo_joint">
-    <origin xyz="0.15 0 .1" rpy="0 0 0"/>
-    <child link="hokuyo"/>
-    <parent link="chassis"/>
-    <axis xyz="1 1 1" rpy="0 0 0"/>
-  </joint>
-  <gazebo reference="left_wheel">
-      <material>Gazebo/Yellow</material>
-  </gazebo>
-  <gazebo reference="right_wheel">
-      <material>Gazebo/Yellow</material>
-  </gazebo>
-  <gazebo reference="chassis">
-      <material>Gazebo/Green</material>
-  </gazebo>
-    <gazebo reference="camera">
-        <material>Gazebo/Red</material>
+ </link>
+     <joint type="continuous" name="left_wheel_hinge">
+       <origin xyz="0.0 0.22 0" rpy="0 0 0"/>
+       <child link="left_wheel"/>
+       <parent link="chassis"/>
+       <axis xyz="0 1 0" rpy="0 0 0"/>
+       <limit effort="10000" velocity="1000"/>
+       <dynamics damping="1.0" friction="1.0"/>
+     </joint>
+      <link name='right_wheel'>
+        <pose>0 0.0 0 0 0 0</pose>
+        <inertial>
+          <mass value="3.0"/>
+          <origin xyz="0.0 0 0" rpy=" 0 1.5707 1.5707"/>
+          <inertia
+              ixx="0.1" ixy="0" ixz="0"
+              iyy="0.1" iyz="0"
+              izz="0.1"/>
+        </inertial>
+        <collision name='right_wheel_collision'>
+          <origin xyz="0 0 0" rpy=" 0 1.5707 1.5707"/>
+          <geometry>
+            <cylinder radius=".08" length="0.025"/>
+          </geometry>
+        </collision>
+        <visual name='right_wheel_visual'>
+          <origin xyz="0 0 0" rpy=" 0 1.5707 1.5707"/>
+          <geometry>
+            <cylinder radius=".08" length="0.025"/>
+        </geometry>
+        </visual>
+     </link>
+     <joint type="continuous" name="right_wheel_hinge">
+      <origin xyz=".0 -0.22 0" rpy="0 0 0"/>
+      <child link="right_wheel"/>
+      <parent link="chassis"/>
+      <axis xyz="0 1 0" rpy="0 0 0"/>
+      <limit effort="10000" velocity="1000"/>
+      <dynamics damping="1.0" friction="1.0"/>
+    </joint>
+    <link name='hokuyo'>
+       <pose>0.0 0 .0 0 0 0</pose>
+       <inertial>
+         <mass value="1e-5"/>
+         <origin xyz="0 0 0" rpy=" 0 0 0"/>
+         <inertia
+             ixx="1e-6" ixy="0" ixz="0"
+             iyy="1e-6" iyz="0"
+             izz="1e-6"/>
+       </inertial>
+       <collision name='hokuyo_collision'>
+         <origin xyz="0 0 0" rpy=" 0 0 0"/>
+         <geometry>
+           <box size=".1 .1 .1"/>
+         </geometry>
+       </collision>
+       <visual name='hokuyo_visual'>
+         <origin xyz="0 0 0" rpy=" 0 0 0"/>
+         <geometry>
+           <mesh filename="package://my_robot/meshes/hokuyo.dae"/>
+         </geometry>
+       </visual>
+     </link>
+     <joint type="fixed" name="hokuyo_joint">
+       <origin xyz="0.1 0 .08" rpy="0 0 0"/>
+       <child link="hokuyo"/>
+       <parent link="chassis"/>
+       <axis xyz="1 1 1" rpy="0 0 0"/>
+     </joint>
+     <link name='camera'>
+       <pose> 0.0 0 0 0 0 0</pose>
+       <inertial>
+         <mass value=".1"/>
+         <origin xyz="0 0 0" rpy=" 0 0 0"/>
+         <inertia
+             ixx="1e-6" ixy="0" ixz="0"
+             iyy="1e-6" iyz="0"
+             izz="1e-6"/>
+       </inertial>
+       <collision name='camera_collision'>
+         <origin xyz="0 0 0" rpy=" 0 0 0"/>
+         <geometry>
+           <box size=".03 .03 .03"/>
+         </geometry>
+       </collision>
+       <visual name='camera_visual'>
+         <origin xyz="0 0 0" rpy=" 0 0 0"/>
+         <geometry>
+           <box size=".03 .03 .03"/>
+         </geometry>
+       </visual>
+     </link>
+    <joint type="fixed" name="camera_joint">
+        <origin xyz="0.14 0 0.03" rpy="0 0 0"/>
+        <child link="camera"/>
+        <parent link="chassis"/>
+        <axis xyz="1 1 1" rpy="0 0 0"/>
+    </joint>
+    <gazebo reference="left_wheel">
+        <material>Gazebo/Yellow</material>
     </gazebo>
+    <gazebo reference="right_wheel">
+        <material>Gazebo/Yellow</material>
+    </gazebo>
+    <gazebo reference="chassis">
+        <material>Gazebo/Green</material>
+    </gazebo>
+      <gazebo reference="camera">
+          <material>Gazebo/Red</material>
+      </gazebo>
 </robot>
