Commit message: feat: Add RGB-D camera to .gazebo and .xacro

File: project_4/catkin_ws/src/my_robot/urdf/my_robot.xacro (robot description, xacro)
@@ -170,4 +170,11 @@
        </visual>
      </link>
+    <joint name="camera_optical_joint" type="fixed">
+      <origin xyz="0 0 0" rpy="-1.5707 0 -1.5707"/>
+      <parent link="camera"/>
+      <child link="camera_link_optical"/>
+    </joint>
+    <link name="camera_link_optical">
+    </link>
     <joint type="fixed" name="camera_joint">
         <origin xyz="0.14 0 0.03" rpy="0 0 0"/>
